File: hardware/board.sch (EAGLE design)
At the start: 46 parts, among them IC1 0915BM15A0001, J1 U.FL, U3 BLE113-A, X1 24MHz 8pF 10ppm -20C +70C, X3 MINI-USB-UX60-MB-5ST

Commit message: JDBP changes: BOM adjustments, microUSB
Parts:
- removed ALT.PWR: (no value), pinhead:PINHD-1X2
- removed R4, R9: (no value), rcl:R-US_R0402
- removed X3: MINI-USB-UX60-MB-5ST, con-hirose:MINI-USB-UX60-MB-5ST
- BLE113-DEBUG, CC1110-DEBUG: value CC-DEBUG-PWR -> 20021121-00010C4LF
- C11: device rcl:C-USC0805K -> rcl:C-USC1206
- C14, C2, C3: value 4.7uF -> 10uF; device rcl:C-USC0603K -> rcl:C-USC1206
- C4: value 10 uF -> 10uF; device rcl:C-EUC0805K -> rcl:C-USC1206
- CC1110: value CC1110 -> CC1110F32RHHR
- IC1: value 0915BM15A0001 -> 0915BM15A0001E
- J1: value U.FL -> MF-CON-MICROUSB-RIGHT; device SparkFun-Connectors:U.FL -> MF_Connectors:USB_MICRO_RIGHT
- JP1: value M02-JST-2MM-SMT -> S2B-PH-SM4-TB(LF)(SN)
- LED2, LED5: value blue -> red
- R11, R12, R13, R7: value 470 ohms -> 470
- R2: value 330 -> 470
- U1: value (none) -> MCP73831T
- U3: value BLE113-A -> BLE113-A-M256K
- VREG: value LM3671 -> LM3671MF-3.3/NOPB
Connections:
- removed net N$12: ANT1.1, R9.2
- removed net N$9: J1.SIGNAL, R4.1
- net GND: now also J1.GND, J1.SLD; no longer ALT.PWR.1, J1.GND@0, J1.GND@1, X3.5
- net N$10: now also ANT1.1; no longer R4.2, R9.1
- net VIN_USB: now also J1.5V; no longer ALT.PWR.2, X3.1
Other:
- moved on the sheet: ANT1

Commit message: More trace and part packing; DRC approvals
Parts:
- C9: device rcl:C-EUC0402K -> rcl:C-EUC0402
Changed lines of the file:
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@@
 <part name="R3" library="rcl" deviceset="R-US_" device="R0402" value="56kOhm ± 1%"/>
 <part name="GND17" library="supply1" deviceset="GND" device=""/>
-<part name="C9" library="rcl" deviceset="C-EU" device="C0402K" value="1uF"/>
+<part name="C9" library="rcl" deviceset="C-EU" device="C0402" value="1uF"/>
 <part name="GND18" library="supply1" deviceset="GND" device=""/>
 <part name="IC1" library="parts" deviceset="0915BM15A0001" device="" value="0915BM15A0001E"/>

Commit message: More changes
Parts:
- removed BLE113-DEBUG, CC1110-DEBUG: 20021121-00010C4LF, parts:CC-DEBUG-PWR
- removed C13: 0.1uF, rcl:C-EUC0402
- removed C14: 10uF, rcl:C-USC1206
- removed LED4: green, led:LEDSML0603
- removed LED5: red, led:LEDSML0603
- removed R11, R7: 470, rcl:R-US_R0402
- added C15: 0.1uF, rcl:C-EUC0402
- added C20: (no value), rcl:C-EUC0402
- added L2: (no value), rcl:R-US_R0402
- added TC1, TC2: TC2050-IDC-NL, TagConnect:TC2050-IDC-NL
- ANT1: device discrete:ANTENNA -> board:ANTENNASMT
- C1: value 0.1uF -> 10uF; device rcl:C-EUC0402 -> rcl:C-USC1206
- C11: value 10uF -> 0.1uF; device rcl:C-USC1206 -> rcl:C-EUC0402
- C7: value 0.1uF -> 1uF
- C9: value 1uF -> 0.1uF
- IC1: value 0915BM15A0001E -> 0433BM15A0001
- R2: value 470 -> 56kOhm ± 1%
- R3: value 56kOhm ± 1% -> 470
- renumbered R12 to R4, R13 to R5
Connections:
- removed net N$24: LED4.A, R7.1
- removed net N$25: LED5.A, R11.1
- new net N$1: ANT1.1, L2.2
- net DC: now also TC1.5; no longer CC1110-DEBUG.DC
- net DC_BLE: now also TC2.5; no longer BLE113-DEBUG.DC
- net DD: now also TC1.7; no longer CC1110-DEBUG.DD
- net DD_BLE: now also TC2.7; no longer BLE113-DEBUG.DD
- net GND: now also C15.2, C20.2, C7.1, C9.2, R2.1, TC1.1, TC2.1; no longer BLE113-DEBUG.GND, C13.2, C14.2, C7.2, C9.1, CC1110-DEBUG.GND, LED4.C, LED5.C, R3.1
- net MISO: now also TC1.2; no longer BLE113-DEBUG.MISO, CC1110-DEBUG.MISO
- net MOSI: now also TC1.6; no longer BLE113-DEBUG.MOSI, CC1110-DEBUG.MOSI
- net N$10: now also C20.1, L2.1; no longer ANT1.1
- net N$14: now also R2.2; no longer R3.2
- net N$18: now also C7.2; no longer C9.2
- net N$4: now also R3.2; no longer R2.2
- net P0_0: no longer R7.2
- net P0_1: no longer R11.2
- net RESET: now also TC1.8, TC2.8; no longer BLE113-DEBUG.RES, CC1110-DEBUG.RES
- net SCK: now also TC1.10; no longer BLE113-DEBUG.SCK, CC1110-DEBUG.SCK
- net SSN: now also TC1.9; no longer BLE113-DEBUG.SSN, CC1110-DEBUG.SSN
- net V+: now also C1.1; no longer C14.1
- net VDD: now also C15.1, C9.1, TC1.3, TC2.3; no longer BLE113-DEBUG.3V3_SENS, C1.1, C13.1, C7.1, CC1110-DEBUG.3V3_SENS
- net VIN_USB: now also R3.1; no longer R2.1
Other:
- note added: "CC1110"
- moved on the sheet: C1, C11, C12, C7, C9, R2, R3
